File: bb1/teensy.sch (KiCad schematic (older format))
At the start: 29 parts, among them J1 USB-MICRO-B-SHIELDED, P4 USB_POWER, P6 CORTEX_DEBUG, SW1 RESET, SW2 PROGRAM, U7 LP38691, U8 MK20DX256VLH7, U9 MKL02Z32VFG4, X1 CRYSTAL_SMD, Y2 32kHz

Commit message: Continued work on the PCB. Lots of footprint work.
Parts:
- removed SW1: RESET, bb:SWITCH_SMD_3x6, symbol SW_PUSH
- added SJ3: SOLDER_JUMPER, symbol SOLDER_JUMPER
- Y2: footprint Crystals:Crystal_Watch -> bb:Crystal_Watch_6mm
- renumbered SW2 to SW1
Connections:
- net RESET: now also SJ3.2
- net at SW1.1, U9.18 (PTB2): now also SJ3.1
Changed lines of the file:
@@
 $EndComp
 $Comp
-L GND #PWR040
+L GND #PWR57
 U 1 1 5658E841
 P 6850 5300
-F 0 "#PWR040" H 6850 5050 50  0001 C CNN
+F 0 "#PWR57" H 6850 5050 50  0001 C CNN
 F 1 "GND" H 6850 5150 50  0000 C CNN
 F 2 "" H 6850 5300 60  0000 C CNN
@@
 $EndComp
 $Comp
-L +3.3V #PWR041
+L +3.3V #PWR53
 U 1 1 5658ECFF
 P 1600 3450
-F 0 "#PWR041" H 1600 3300 50  0001 C CNN
+F 0 "#PWR53" H 1600 3300 50  0001 C CNN
 F 1 "+3.3V" H 1600 3590 50  0000 C CNN
 F 2 "" H 1600 3450 60  0000 C CNN
@@
 $EndComp
 $Comp
-L GND #PWR042
+L GND #PWR55
 U 1 1 5658ED8D
 P 1400 4050
-F 0 "#PWR042" H 1400 3800 50  0001 C CNN
+F 0 "#PWR55" H 1400 3800 50  0001 C CNN
 F 1 "GND" H 1400 3900 50  0000 C CNN
 F 2 "" H 1400 4050 60  0000 C CNN
@@
 RESET
 $Comp
-L SW_PUSH SW2
+L SW_PUSH SW1
 U 1 1 5658EF9A
 P 3750 4900
-F 0 "SW2" H 3900 5010 50  0000 C CNN
+F 0 "SW1" H 3900 5010 50  0000 C CNN
 F 1 "PROGRAM" H 3750 4820 50  0000 C CNN
 F 2 "bb:SWITCH_SMD_3x6" H 3750 4900 60  0001 C CNN
@@
 $EndComp
 $Comp
-L GND #PWR043
+L GND #PWR56
 U 1 1 5658F088
-P 4400 5000
-F 0 "#PWR043" H 4400 4750 50  0001 C CNN
-F 1 "GND" H 4400 4850 50  0000 C CNN
-F 2 "" H 4400 5000 60  0000 C CNN
-F 3 "" H 4400 5000 60  0000 C CNN
-	1    4400 5000
+P 4100 4950
+F 0 "#PWR56" H 4100 4700 50  0001 C CNN
+F 1 "GND" H 4100 4800 50  0000 C CNN
+F 2 "" H 4100 4950 60  0000 C CNN
+F 3 "" H 4100 4950 60  0000 C CNN
+	1    4100 4950
 	1    0    0    -1
 $EndComp
@@
 $EndComp
 $Comp
-L +3.3V #PWR044
+L +3.3V #PWR58
 U 1 1 56590BBB
 P 1600 5850
-F 0 "#PWR044" H 1600 5700 50  0001 C CNN
+F 0 "#PWR58" H 1600 5700 50  0001 C CNN
 F 1 "+3.3V" H 1600 5990 50  0000 C CNN
 F 2 "" H 1600 5850 60  0000 C CNN
@@
 NoConn ~ 1850 6300
 $Comp
-L GND #PWR045
+L GND #PWR48
 U 1 1 565927D7
 P 1700 2150
-F 0 "#PWR045" H 1700 1900 50  0001 C CNN
+F 0 "#PWR48" H 1700 1900 50  0001 C CNN
 F 1 "GND" H 1700 2000 50  0000 C CNN
 F 2 "" H 1700 2150 60  0000 C CNN
@@
 $EndComp
 $Comp
-L +3.3V #PWR046
+L +3.3V #PWR43
 U 1 1 56596469
 P 6600 1400
-F 0 "#PWR046" H 6600 1250 50  0001 C CNN
+F 0 "#PWR43" H 6600 1250 50  0001 C CNN
 F 1 "+3.3V" H 6600 1540 50  0000 C CNN
 F 2 "" H 6600 1400 60  0000 C CNN
@@
 $EndComp
 $Comp
-L GND #PWR047
+L GND #PWR47
 U 1 1 565968B4
 P 5900 1900
-F 0 "#PWR047" H 5900 1650 50  0001 C CNN
+F 0 "#PWR47" H 5900 1650 50  0001 C CNN
 F 1 "GND" H 5900 1750 50  0000 C CNN
 F 2 "" H 5900 1900 60  0000 C CNN
@@
 $EndComp
 $Comp
-L GND #PWR048
+L GND #PWR50
 U 1 1 56598327
 P 5300 3300
-F 0 "#PWR048" H 5300 3050 50  0001 C CNN
+F 0 "#PWR50" H 5300 3050 50  0001 C CNN
 F 1 "GND" H 5300 3150 50  0000 C CNN
 F 2 "" H 5300 3300 60  0000 C CNN
@@
 F 0 "Y2" H 6800 3500 50  0000 C CNN
 F 1 "32kHz" H 6800 3300 50  0000 C CNN
-F 2 "Crystals:Crystal_Watch" H 6800 3400 60  0001 C CNN
+F 2 "bb:Crystal_Watch_6mm" H 6800 3400 60  0001 C CNN
 F 3 "" H 6800 3400 60  0000 C CNN
 	1    6800 3400
@@
 $EndComp
 $Comp
-L GND #PWR049
+L GND #PWR45
 U 1 1 565A6A4F
 P 3550 1700
-F 0 "#PWR049" H 3550 1450 50  0001 C CNN
+F 0 "#PWR45" H 3550 1450 50  0001 C CNN
 F 1 "GND" H 3550 1550 50  0000 C CNN
 F 2 "" H 3550 1700 60  0000 C CNN
@@
 $EndComp
 $Comp
-L +5V #PWR050
+L +5V #PWR41
 U 1 1 565A6A86
 P 2900 1250
-F 0 "#PWR050" H 2900 1100 50  0001 C CNN
+F 0 "#PWR41" H 2900 1100 50  0001 C CNN
 F 1 "+5V" H 2900 1390 50  0000 C CNN
 F 2 "" H 2900 1250 60  0000 C CNN
@@
 	1700 4300 1100 4300
 Wire Wire Line
-	4050 4900 4400 4900
-Wire Wire Line
-	4400 4600 4400 5000
+	4050 4900 4100 4900
 Wire Wire Line
 	3200 5000 3200 5200
@@
 	7050 2600 6900 2600
 Wire Wire Line
-	6900 2600 6900 2700
+	6900 2700 6900 2600
 Connection ~ 6900 2700
 Wire Wire Line
@@
 	3950 1350 4250 1350
 $Comp
-L +3.3V #PWR051
+L +3.3V #PWR42
 U 1 1 565A6D4A
 P 4250 1250
-F 0 "#PWR051" H 4250 1100 50  0001 C CNN
+F 0 "#PWR42" H 4250 1100 50  0001 C CNN
 F 1 "+3.3V" H 4250 1390 50  0000 C CNN
 F 2 "" H 4250 1250 60  0000 C CNN
@@
 	3550 1600 3550 1700
 $Comp
-L GND #PWR052
+L GND #PWR46
 U 1 1 565A70D1
 P 4100 1700
-F 0 "#PWR052" H 4100 1450 50  0001 C CNN
+F 0 "#PWR46" H 4100 1450 50  0001 C CNN
 F 1 "GND" H 4100 1550 50  0000 C CNN
 F 2 "" H 4100 1700 60  0000 C CNN
@@
 	3000 1650 3000 1700
 $Comp
-L GND #PWR053
+L GND #PWR44
 U 1 1 565AC891
 P 3000 1700
-F 0 "#PWR053" H 3000 1450 50  0001 C CNN
+F 0 "#PWR44" H 3000 1450 50  0001 C CNN
 F 1 "GND" H 3000 1550 50  0000 C CNN
 F 2 "" H 3000 1700 60  0000 C CNN
@@
 $EndComp
 $Comp
-L +5V #PWR054
+L +5V #PWR39
 U 1 1 565AEF07
 P 2300 750
-F 0 "#PWR054" H 2300 600 50  0001 C CNN
+F 0 "#PWR39" H 2300 600 50  0001 C CNN
 F 1 "+5V" H 2300 890 50  0000 C CNN
 F 2 "" H 2300 750 60  0000 C CNN
@@
 $EndComp
 $Comp
-L GND #PWR055
+L GND #PWR40
 U 1 1 565B08A1
 P 1500 1150
-F 0 "#PWR055" H 1500 900 50  0001 C CNN
+F 0 "#PWR40" H 1500 900 50  0001 C CNN
 F 1 "GND" H 1500 1000 50  0000 C CNN
 F 2 "" H 1500 1150 60  0000 C CNN
@@
 	8250 2450 8600 2450
 $Comp
-L GND #PWR056
+L GND #PWR49
 U 1 1 565BDF2E
 P 10200 2600
-F 0 "#PWR056" H 10200 2350 50  0001 C CNN
+F 0 "#PWR49" H 10200 2350 50  0001 C CNN
 F 1 "GND" H 10200 2450 50  0000 C CNN
 F 2 "" H 10200 2600 60  0000 C CNN
@@
 Wire Wire Line
 	8250 5300 8600 5300
-Wire Wire Line
-	3150 4200 3150 4600
-Wire Wire Line
-	3150 4600 3450 4600
-Connection ~ 3150 4200
-$Comp
-L SW_PUSH SW1
-U 1 1 565C8555
-P 3750 4600
-F 0 "SW1" H 3900 4710 50  0000 C CNN
-F 1 "RESET" H 3750 4520 50  0000 C CNN
-F 2 "bb:SWITCH_SMD_3x6" H 3750 4600 60  0001 C CNN
-F 3 "" H 3750 4600 60  0000 C CNN
-	1    3750 4600
-	1    0    0    -1
-$EndComp
-Wire Wire Line
-	4050 4600 4400 4600
-Connection ~ 4400 4900
 $Comp
 L CONN_01X02 P4
@@
 NoConn ~ 1800 4300
 $Comp
-L +3.3V #PWR057
+L +3.3V #PWR51
 U 1 1 567B1DAE
 P 5750 3300
-F 0 "#PWR057" H 5750 3150 50  0001 C CNN
+F 0 "#PWR51" H 5750 3150 50  0001 C CNN
 F 1 "+3.3V" H 5750 3440 50  0000 C CNN
 F 2 "" H 5750 3300 60  0000 C CNN
@@
 Connection ~ 5750 3350
 $Comp
-L GND #PWR058
+L GND #PWR54
 U 1 1 567B220D
 P 5750 3650
-F 0 "#PWR058" H 5750 3400 50  0001 C CNN
+F 0 "#PWR54" H 5750 3400 50  0001 C CNN
 F 1 "GND" H 5750 3500 50  0000 C CNN
 F 2 "" H 5750 3650 60  0000 C CNN
@@
 Connection ~ 5200 2250
 $Comp
-L PWR_FLAG #FLG059
+L PWR_FLAG #FLG2
 U 1 1 567B5BB9
 P 5550 2200
-F 0 "#FLG059" H 5550 2295 50  0001 C CNN
+F 0 "#FLG2" H 5550 2295 50  0001 C CNN
 F 1 "PWR_FLAG" H 5550 2380 50  0000 C CNN
 F 2 "" H 5550 2200 60  0000 C CNN
@@
 	6600 3200 6600 3300
 $Comp
-L GND #PWR060
+L GND #PWR52
 U 1 1 568579A5
 P 6600 3300
-F 0 "#PWR060" H 6600 3050 50  0001 C CNN
+F 0 "#PWR52" H 6600 3050 50  0001 C CNN
 F 1 "GND" H 6600 3150 50  0000 C CNN
 F 2 "" H 6600 3300 60  0000 C CNN
@@
 Connection ~ 1600 6150
 $Comp
-L GND #PWR061
+L GND #PWR59
 U 1 1 56858A76
 P 1100 6250
-F 0 "#PWR061" H 1100 6000 50  0001 C CNN
+F 0 "#PWR59" H 1100 6000 50  0001 C CNN
 F 1 "GND" H 1100 6100 50  0000 C CNN
 F 2 "" H 1100 6250 60  0000 C CNN
@@
 Wire Wire Line
 	1350 3600 1350 3650
+$Comp
+L SOLDER_JUMPER SJ3
+U 1 1 56652374
+P 3350 4550
+F 0 "SJ3" V 3430 4550 50  0000 C CNN
+F 1 "SOLDER_JUMPER" V 3250 4550 50  0000 C CNN
+F 2 "" H 3350 4550 60  0000 C CNN
+F 3 "" H 3350 4550 60  0000 C CNN
+	1    3350 4550
+	1    0    0    1
+$EndComp
+Wire Wire Line
+	3350 4300 3350 4200
+Connection ~ 3350 4200
+Wire Wire Line
+	3350 4800 3350 4900
+Connection ~ 3350 4900
+Wire Wire Line
+	4100 4900 4100 4950
 $EndSCHEMATC

Commit message: Finalized v1 revA
 - Added BNO055
 - Fixed SOIC8 pattern
 - Replaced phoenix connectors by a 20 pol
 - Many fine tuning/cosmetic adjustments
 - Sent files to manufacturing. Will tag this commit.
Parts:
- SJ3: footprint (none) -> bb:SolderJumper
Changed lines of the file:
@@
 $Descr A4 11693 8268
 encoding utf-8
-Sheet 2 3
+Sheet 2 4
 Title ""
 Date ""
@@
 $EndComp
 $Comp
-L GND #PWR57
+L GND #PWR033
 U 1 1 5658E841
 P 6850 5300
-F 0 "#PWR57" H 6850 5050 50  0001 C CNN
+F 0 "#PWR033" H 6850 5050 50  0001 C CNN
 F 1 "GND" H 6850 5150 50  0000 C CNN
 F 2 "" H 6850 5300 60  0000 C CNN
@@
 $EndComp
 $Comp
-L +3.3V #PWR53
+L +3.3V #PWR034
 U 1 1 5658ECFF
 P 1600 3450
-F 0 "#PWR53" H 1600 3300 50  0001 C CNN
+F 0 "#PWR034" H 1600 3300 50  0001 C CNN
 F 1 "+3.3V" H 1600 3590 50  0000 C CNN
 F 2 "" H 1600 3450 60  0000 C CNN
@@
 $EndComp
 $Comp
-L GND #PWR55
+L GND #PWR035
 U 1 1 5658ED8D
 P 1400 4050
-F 0 "#PWR55" H 1400 3800 50  0001 C CNN
+F 0 "#PWR035" H 1400 3800 50  0001 C CNN
 F 1 "GND" H 1400 3900 50  0000 C CNN
 F 2 "" H 1400 4050 60  0000 C CNN
@@
 $EndComp
 $Comp
-L GND #PWR56
+L GND #PWR036
 U 1 1 5658F088
 P 4100 4950
-F 0 "#PWR56" H 4100 4700 50  0001 C CNN
+F 0 "#PWR036" H 4100 4700 50  0001 C CNN
 F 1 "GND" H 4100 4800 50  0000 C CNN
 F 2 "" H 4100 4950 60  0000 C CNN
@@
 $EndComp
 $Comp
-L +3.3V #PWR58
+L +3.3V #PWR037
 U 1 1 56590BBB
 P 1600 5850
-F 0 "#PWR58" H 1600 5700 50  0001 C CNN
+F 0 "#PWR037" H 1600 5700 50  0001 C CNN
 F 1 "+3.3V" H 1600 5990 50  0000 C CNN
 F 2 "" H 1600 5850 60  0000 C CNN
@@
 NoConn ~ 1850 6300
 $Comp
-L GND #PWR48
+L GND #PWR038
 U 1 1 565927D7
 P 1700 2150
-F 0 "#PWR48" H 1700 1900 50  0001 C CNN
+F 0 "#PWR038" H 1700 1900 50  0001 C CNN
 F 1 "GND" H 1700 2000 50  0000 C CNN
 F 2 "" H 1700 2150 60  0000 C CNN
@@
 $EndComp
 $Comp
-L +3.3V #PWR43
+L +3.3V #PWR039
 U 1 1 56596469
 P 6600 1400
-F 0 "#PWR43" H 6600 1250 50  0001 C CNN
+F 0 "#PWR039" H 6600 1250 50  0001 C CNN
 F 1 "+3.3V" H 6600 1540 50  0000 C CNN
 F 2 "" H 6600 1400 60  0000 C CNN
@@
 $EndComp
 $Comp
-L GND #PWR47
+L GND #PWR040
 U 1 1 565968B4
 P 5900 1900
-F 0 "#PWR47" H 5900 1650 50  0001 C CNN
+F 0 "#PWR040" H 5900 1650 50  0001 C CNN
 F 1 "GND" H 5900 1750 50  0000 C CNN
 F 2 "" H 5900 1900 60  0000 C CNN
@@
 $EndComp
 $Comp
-L GND #PWR50
+L GND #PWR041
 U 1 1 56598327
 P 5300 3300
-F 0 "#PWR50" H 5300 3050 50  0001 C CNN
+F 0 "#PWR041" H 5300 3050 50  0001 C CNN
 F 1 "GND" H 5300 3150 50  0000 C CNN
 F 2 "" H 5300 3300 60  0000 C CNN
@@
 $EndComp
 $Comp
-L GND #PWR45
+L GND #PWR042
 U 1 1 565A6A4F
 P 3550 1700
-F 0 "#PWR45" H 3550 1450 50  0001 C CNN
+F 0 "#PWR042" H 3550 1450 50  0001 C CNN
 F 1 "GND" H 3550 1550 50  0000 C CNN
 F 2 "" H 3550 1700 60  0000 C CNN
@@
 $EndComp
 $Comp
-L +5V #PWR41
+L +5V #PWR043
 U 1 1 565A6A86
 P 2900 1250
-F 0 "#PWR41" H 2900 1100 50  0001 C CNN
+F 0 "#PWR043" H 2900 1100 50  0001 C CNN
 F 1 "+5V" H 2900 1390 50  0000 C CNN
 F 2 "" H 2900 1250 60  0000 C CNN
@@
 	7050 2600 6900 2600
 Wire Wire Line
-	6900 2700 6900 2600
+	6900 2600 6900 2700
 Connection ~ 6900 2700
 Wire Wire Line
@@
 	3950 1350 4250 1350
 $Comp
-L +3.3V #PWR42
+L +3.3V #PWR044
 U 1 1 565A6D4A
 P 4250 1250
-F 0 "#PWR42" H 4250 1100 50  0001 C CNN
+F 0 "#PWR044" H 4250 1100 50  0001 C CNN
 F 1 "+3.3V" H 4250 1390 50  0000 C CNN
 F 2 "" H 4250 1250 60  0000 C CNN
@@
 	3550 1600 3550 1700
 $Comp
-L GND #PWR46
+L GND #PWR045
 U 1 1 565A70D1
 P 4100 1700
-F 0 "#PWR46" H 4100 1450 50  0001 C CNN
+F 0 "#PWR045" H 4100 1450 50  0001 C CNN
 F 1 "GND" H 4100 1550 50  0000 C CNN
 F 2 "" H 4100 1700 60  0000 C CNN
@@
 	3000 1650 3000 1700
 $Comp
-L GND #PWR44
+L GND #PWR046
 U 1 1 565AC891
 P 3000 1700
-F 0 "#PWR44" H 3000 1450 50  0001 C CNN
+F 0 "#PWR046" H 3000 1450 50  0001 C CNN
 F 1 "GND" H 3000 1550 50  0000 C CNN
 F 2 "" H 3000 1700 60  0000 C CNN
@@
 $EndComp
 $Comp
-L +5V #PWR39
+L +5V #PWR047
 U 1 1 565AEF07
 P 2300 750
-F 0 "#PWR39" H 2300 600 50  0001 C CNN
+F 0 "#PWR047" H 2300 600 50  0001 C CNN
 F 1 "+5V" H 2300 890 50  0000 C CNN
 F 2 "" H 2300 750 60  0000 C CNN
@@
 $EndComp
 $Comp
-L GND #PWR40
+L GND #PWR048
 U 1 1 565B08A1
 P 1500 1150
-F 0 "#PWR40" H 1500 900 50  0001 C CNN
+F 0 "#PWR048" H 1500 900 50  0001 C CNN
 F 1 "GND" H 1500 1000 50  0000 C CNN
 F 2 "" H 1500 1150 60  0000 C CNN
@@
 	8250 2450 8600 2450
 $Comp
-L GND #PWR49
+L GND #PWR049
 U 1 1 565BDF2E
 P 10200 2600
-F 0 "#PWR49" H 10200 2350 50  0001 C CNN
+F 0 "#PWR049" H 10200 2350 50  0001 C CNN
 F 1 "GND" H 10200 2450 50  0000 C CNN
 F 2 "" H 10200 2600 60  0000 C CNN
@@
 NoConn ~ 1800 4300
 $Comp
-L +3.3V #PWR51
+L +3.3V #PWR050
 U 1 1 567B1DAE
 P 5750 3300
-F 0 "#PWR51" H 5750 3150 50  0001 C CNN
+F 0 "#PWR050" H 5750 3150 50  0001 C CNN
 F 1 "+3.3V" H 5750 3440 50  0000 C CNN
 F 2 "" H 5750 3300 60  0000 C CNN
@@
 Connection ~ 5750 3350
 $Comp
-L GND #PWR54
+L GND #PWR051
 U 1 1 567B220D
 P 5750 3650
-F 0 "#PWR54" H 5750 3400 50  0001 C CNN
+F 0 "#PWR051" H 5750 3400 50  0001 C CNN
 F 1 "GND" H 5750 3500 50  0000 C CNN
 F 2 "" H 5750 3650 60  0000 C CNN
@@
 Connection ~ 5200 2250
 $Comp
-L PWR_FLAG #FLG2
+L PWR_FLAG #FLG052
 U 1 1 567B5BB9
 P 5550 2200
-F 0 "#FLG2" H 5550 2295 50  0001 C CNN
+F 0 "#FLG052" H 5550 2295 50  0001 C CNN
 F 1 "PWR_FLAG" H 5550 2380 50  0000 C CNN
 F 2 "" H 5550 2200 60  0000 C CNN
@@
 	6600 3200 6600 3300
 $Comp
-L GND #PWR52
+L GND #PWR053
 U 1 1 568579A5
 P 6600 3300
-F 0 "#PWR52" H 6600 3050 50  0001 C CNN
+F 0 "#PWR053" H 6600 3050 50  0001 C CNN
 F 1 "GND" H 6600 3150 50  0000 C CNN
 F 2 "" H 6600 3300 60  0000 C CNN
@@
 Connection ~ 1600 6150
 $Comp
-L GND #PWR59
+L GND #PWR054
 U 1 1 56858A76
 P 1100 6250
-F 0 "#PWR59" H 1100 6000 50  0001 C CNN
+F 0 "#PWR054" H 1100 6000 50  0001 C CNN
 F 1 "GND" H 1100 6100 50  0000 C CNN
 F 2 "" H 1100 6250 60  0000 C CNN
@@
 F 0 "SJ3" V 3430 4550 50  0000 C CNN
 F 1 "SOLDER_JUMPER" V 3250 4550 50  0000 C CNN
-F 2 "" H 3350 4550 60  0000 C CNN
+F 2 "bb:SolderJumper" H 3350 4550 60  0001 C CNN
 F 3 "" H 3350 4550 60  0000 C CNN
 	1    3350 4550
