File: hardware-v1/nmea.sch (KiCad schematic (older format))
At the start: 24 parts, among them P1 CONN_01X20, U10 MCP2562, U11 SN65C1168E, U12 INA219

Commit message: re-annotate schematic
Parts:
- gave numbers to parts that had none: 2
Changed lines of the file:
@@
 $EndComp
 $Comp
-L GND #PWR055
+L GND #PWR61
 U 1 1 5660859F
 P 3250 5850
-F 0 "#PWR055" H 3250 5600 50  0001 C CNN
+F 0 "#PWR61" H 3250 5600 50  0001 C CNN
 F 1 "GND" H 3250 5700 50  0000 C CNN
 F 2 "" H 3250 5850 60  0000 C CNN
@@
 $EndComp
 $Comp
-L +3.3V #PWR056
+L +3.3V #PWR52
 U 1 1 5661817C
 P 3500 2200
-F 0 "#PWR056" H 3500 2050 50  0001 C CNN
+F 0 "#PWR52" H 3500 2050 50  0001 C CNN
 F 1 "+3.3V" H 3500 2340 50  0000 C CNN
 F 2 "" H 3500 2200 60  0000 C CNN
@@
 $EndComp
 $Comp
-L GND #PWR057
+L GND #PWR51
 U 1 1 5661CF45
 P 1900 2150
-F 0 "#PWR057" H 1900 1900 50  0001 C CNN
+F 0 "#PWR51" H 1900 1900 50  0001 C CNN
 F 1 "GND" H 1900 2000 50  0000 C CNN
 F 2 "" H 1900 2150 60  0000 C CNN
@@
 $EndComp
 $Comp
-L +5V #PWR058
+L +5V #PWR50
 U 1 1 5661EB70
 P 1600 1700
-F 0 "#PWR058" H 1600 1550 50  0001 C CNN
+F 0 "#PWR50" H 1600 1550 50  0001 C CNN
 F 1 "+5V" H 1600 1840 50  0000 C CNN
 F 2 "" H 1600 1700 60  0000 C CNN
@@
 $EndComp
 $Comp
-L GND #PWR059
+L GND #PWR54
 U 1 1 5663157A
 P 3400 2550
-F 0 "#PWR059" H 3400 2300 50  0001 C CNN
+F 0 "#PWR54" H 3400 2300 50  0001 C CNN
 F 1 "GND" H 3400 2400 50  0000 C CNN
 F 2 "" H 3400 2550 60  0000 C CNN
@@
 $EndComp
 $Comp
-L GND #PWR060
+L GND #PWR53
 U 1 1 56633AB1
 P 1600 2250
-F 0 "#PWR060" H 1600 2000 50  0001 C CNN
+F 0 "#PWR53" H 1600 2000 50  0001 C CNN
 F 1 "GND" H 1600 2100 50  0000 C CNN
 F 2 "" H 1600 2250 60  0000 C CNN
@@
 $EndComp
 $Comp
-L GND #PWR062
+L GND #PWR62
 U 1 1 5671B320
 P 3250 6450
-F 0 "#PWR062" H 3250 6200 50  0001 C CNN
+F 0 "#PWR62" H 3250 6200 50  0001 C CNN
 F 1 "GND" H 3250 6300 50  0000 C CNN
 F 2 "" H 3250 6450 60  0000 C CNN
@@
 $EndComp
 $Comp
-L GND #PWR063
+L GND #PWR63
 U 1 1 5671D29F
 P 3250 7050
-F 0 "#PWR063" H 3250 6800 50  0001 C CNN
+F 0 "#PWR63" H 3250 6800 50  0001 C CNN
 F 1 "GND" H 3250 6900 50  0000 C CNN
 F 2 "" H 3250 7050 60  0000 C CNN
@@
 ANALOG3
 $Comp
-L +12V #PWR064
+L +12V #PWR56
 U 1 1 567F4FFA
 P 8250 3800
-F 0 "#PWR064" H 8250 3650 50  0001 C CNN
+F 0 "#PWR56" H 8250 3650 50  0001 C CNN
 F 1 "+12V" H 8250 3940 50  0000 C CNN
 F 2 "" H 8250 3800 60  0000 C CNN
@@
 $EndComp
 $Comp
-L GND #PWR065
+L GND #PWR59
 U 1 1 56805BCC
 P 2250 5100
-F 0 "#PWR065" H 2250 4850 50  0001 C CNN
+F 0 "#PWR59" H 2250 4850 50  0001 C CNN
 F 1 "GND" H 2250 4950 50  0000 C CNN
 F 2 "" H 2250 5100 60  0000 C CNN
@@
 $EndComp
 $Comp
-L PWR_FLAG #FLG066
+L PWR_FLAG #FLG3
 U 1 1 568074D6
 P 7900 3850
-F 0 "#FLG066" H 7900 3945 50  0001 C CNN
+F 0 "#FLG3" H 7900 3945 50  0001 C CNN
 F 1 "PWR_FLAG" H 7900 4030 50  0000 C CNN
 F 2 "" H 7900 3850 60  0000 C CNN
@@
 $EndComp
 $Comp
-L +3.3V #PWR067
+L +3.3V #PWR57
 U 1 1 56699F39
 P 2700 4400
-F 0 "#PWR067" H 2700 4250 50  0001 C CNN
+F 0 "#PWR57" H 2700 4250 50  0001 C CNN
 F 1 "+3.3V" H 2700 4540 50  0000 C CNN
 F 2 "" H 2700 4400 60  0000 C CNN
@@
 $EndComp
 $Comp
-L GND #PWR068
+L GND #PWR58
 U 1 1 5669B7A7
 P 4500 5000
-F 0 "#PWR068" H 4500 4750 50  0001 C CNN
+F 0 "#PWR58" H 4500 4750 50  0001 C CNN
 F 1 "GND" H 4500 4850 50  0000 C CNN
 F 2 "" H 4500 5000 60  0000 C CNN
@@
 $EndComp
 $Comp
-L +5V #PWR069
+L +5V #PWR47
 U 1 1 5665D00E
 P 8450 1100
-F 0 "#PWR069" H 8450 950 50  0001 C CNN
+F 0 "#PWR47" H 8450 950 50  0001 C CNN
 F 1 "+5V" H 8450 1240 50  0000 C CNN
 F 2 "" H 8450 1100 60  0000 C CNN
@@
 $EndComp
 $Comp
-L GND #PWR070
+L GND #PWR49
 U 1 1 5665D465
 P 8650 1500
-F 0 "#PWR070" H 8650 1250 50  0001 C CNN
+F 0 "#PWR49" H 8650 1250 50  0001 C CNN
 F 1 "GND" H 8650 1350 50  0000 C CNN
 F 2 "" H 8650 1500 60  0000 C CNN
@@
 $EndComp
 $Comp
-L GND #PWR071
+L GND #PWR55
 U 1 1 566617E0
 P 7100 2600
-F 0 "#PWR071" H 7100 2350 50  0001 C CNN
+F 0 "#PWR55" H 7100 2350 50  0001 C CNN
 F 1 "GND" H 7100 2450 50  0000 C CNN
 F 2 "" H 7100 2600 60  0000 C CNN
@@
 $EndComp
 $Comp
-L GND #PWR072
+L GND #PWR48
 U 1 1 5667B0C5
 P 7800 1300
-F 0 "#PWR072" H 7800 1050 50  0001 C CNN
+F 0 "#PWR48" H 7800 1050 50  0001 C CNN
 F 1 "GND" H 7800 1150 50  0000 C CNN
 F 2 "" H 7800 1300 60  0000 C CNN
@@
 Connection ~ 8450 4900
 $Comp
-L GND #PWR073
+L GND #PWR60
 U 1 1 566C9EC9
 P 8450 5800
-F 0 "#PWR073" H 8450 5550 50  0001 C CNN
+F 0 "#PWR60" H 8450 5550 50  0001 C CNN
 F 1 "GND" H 8450 5650 50  0000 C CNN
 F 2 "" H 8450 5800 60  0000 C CNN
@@
 I2C Address: 0x40
 $Comp
-L R R?
+L R R25
 U 1 1 56A28792
 P 2100 4550
-F 0 "R?" V 2180 4550 50  0000 C CNN
+F 0 "R25" V 2180 4550 50  0000 C CNN
 F 1 "10" V 2100 4550 50  0000 C CNN
 F 2 "" V 2030 4550 50  0000 C CNN
@@
 $EndComp
 $Comp
-L R R?
+L R R26
 U 1 1 56A28825
 P 2100 4650
-F 0 "R?" V 2180 4650 50  0000 C CNN
+F 0 "R26" V 2180 4650 50  0000 C CNN
 F 1 "10" V 2100 4650 50  0000 C CNN
 F 2 "" V 2030 4650 50  0000 C CNN
