File: hardware-v1/sensors.sch (KiCad schematic (older format))
At the start: 12 parts, among them U10 BMP280, U11 BNO055

Commit message: Final touches + v1revb sent to oshpark
Parts:
- renumbered C22 to C21, C23 to C22, C24 to C23, C25 to C24, C26 to C25, C27 to C26
Changed lines of the file:
@@
 Connection ~ 1400 1400
 $Comp
-L +3.3V #PWR068
+L +3.3V #PWR067
 U 1 1 566E0C88
 P 1400 1200
-F 0 "#PWR068" H 1400 1050 50  0001 C CNN
+F 0 "#PWR067" H 1400 1050 50  0001 C CNN
 F 1 "+3.3V" H 1400 1340 50  0000 C CNN
 F 2 "" H 1400 1200 60  0000 C CNN
@@
 $EndComp
 $Comp
-L C_Small C25
+L C_Small C24
 U 1 1 566E0C8E
 P 1750 1800
-F 0 "C25" H 1760 1870 50  0000 L CNN
+F 0 "C24" H 1760 1870 50  0000 L CNN
 F 1 ".1uF" H 1760 1720 50  0000 L CNN
 F 2 "Capacitors_SMD:C_0603" H 1750 1800 60  0001 C CNN
@@
 $EndComp
 $Comp
-L C_Small C24
+L C_Small C23
 U 1 1 566E0C95
 P 1400 1800
-F 0 "C24" H 1410 1870 50  0000 L CNN
+F 0 "C23" H 1410 1870 50  0000 L CNN
 F 1 ".1uF" H 1410 1720 50  0000 L CNN
 F 2 "Capacitors_SMD:C_0603" H 1400 1800 60  0001 C CNN
@@
 Connection ~ 1900 2000
 $Comp
-L GND #PWR069
+L GND #PWR068
 U 1 1 566E0CA7
 P 1400 2100
-F 0 "#PWR069" H 1400 1850 50  0001 C CNN
+F 0 "#PWR068" H 1400 1850 50  0001 C CNN
 F 1 "GND" H 1400 1950 50  0000 C CNN
 F 2 "" H 1400 2100 60  0000 C CNN
@@
 	3450 1400 3450 1550
 $Comp
-L GND #PWR070
+L GND #PWR069
 U 1 1 566E0CAF
 P 3450 1550
-F 0 "#PWR070" H 3450 1300 50  0001 C CNN
+F 0 "#PWR069" H 3450 1300 50  0001 C CNN
 F 1 "GND" H 3450 1400 50  0000 C CNN
 F 2 "" H 3450 1550 60  0000 C CNN
@@
 	1550 3250 1800 3250
 $Comp
-L +3.3V #PWR071
+L +3.3V #PWR070
 U 1 1 566E0D0B
 P 1650 3200
-F 0 "#PWR071" H 1650 3050 50  0001 C CNN
+F 0 "#PWR070" H 1650 3050 50  0001 C CNN
 F 1 "+3.3V" H 1650 3340 50  0000 C CNN
 F 2 "" H 1650 3200 60  0000 C CNN
@@
 NoConn ~ 7050 1600
 $Comp
-L GND #PWR072
+L GND #PWR071
 U 1 1 566E19B5
 P 5950 3500
-F 0 "#PWR072" H 5950 3250 50  0001 C CNN
+F 0 "#PWR071" H 5950 3250 50  0001 C CNN
 F 1 "GND" H 5950 3350 50  0000 C CNN
 F 2 "" H 5950 3500 60  0000 C CNN
@@
 	6100 1250 6100 2200
 $Comp
-L +3.3V #PWR073
+L +3.3V #PWR072
 U 1 1 566E28E8
 P 6100 1250
-F 0 "#PWR073" H 6100 1100 50  0001 C CNN
+F 0 "#PWR072" H 6100 1100 50  0001 C CNN
 F 1 "+3.3V" H 6100 1390 50  0000 C CNN
 F 2 "" H 6100 1250 60  0000 C CNN
@@
 $EndComp
 $Comp
-L C_Small C26
+L C_Small C25
 U 1 1 566E32A9
 P 6100 2300
-F 0 "C26" H 6110 2370 50  0000 L CNN
+F 0 "C25" H 6110 2370 50  0000 L CNN
 F 1 ".1uF" H 6110 2220 50  0000 L CNN
 F 2 "Capacitors_SMD:C_0603" H 6100 2300 60  0001 C CNN
@@
 NoConn ~ 7250 2800
 $Comp
-L C_Small C27
+L C_Small C26
 U 1 1 566E365A
 P 7350 3050
-F 0 "C27" H 7360 3120 50  0000 L CNN
+F 0 "C26" H 7360 3120 50  0000 L CNN
 F 1 ".1uF" H 7360 2970 50  0000 L CNN
 F 2 "Capacitors_SMD:C_0603" H 7350 3050 60  0001 C CNN
@@
 Connection ~ 6300 1350
 $Comp
-L C_Small C22
+L C_Small C21
 U 1 1 566E6D3B
 P 6800 1150
-F 0 "C22" H 6810 1220 50  0000 L CNN
+F 0 "C21" H 6810 1220 50  0000 L CNN
 F 1 "6.8nF" H 6810 1070 50  0000 L CNN
 F 2 "Capacitors_SMD:C_0603" H 6800 1150 60  0001 C CNN
@@
 $EndComp
 $Comp
-L C_Small C23
+L C_Small C22
 U 1 1 566E789F
 P 7150 1150
-F 0 "C23" H 7160 1220 50  0000 L CNN
+F 0 "C22" H 7160 1220 50  0000 L CNN
 F 1 "120nF" H 7160 1070 50  0000 L CNN
 F 2 "Capacitors_SMD:C_0603" H 7150 1150 60  0001 C CNN
