File: rgbs.sch (KiCad schematic (older format))
At the start: 10 parts, among them U12 SN74HCT245, U13 N2K_RGB, U14 WIFI_RGB, U15 NMEA_RGB

Commit message: More renaming from bb to kbox
Parts:
- U13, U14, U15: footprint bb:WS2818RGB -> kbox:WS2818RGB
Changed lines of the file:
@@
 EESchema Schematic File Version 2
-LIBS:bb
+LIBS:kbox
 LIBS:power
 LIBS:device
@@
 LIBS:w_device
 LIBS:gsg-symbols
-LIBS:bb1-cache
+LIBS:kbox-cache
 EELAYER 25 0
 EELAYER END
@@
 F 0 "U13" H 3750 3750 60  0000 C CNN
 F 1 "N2K_RGB" H 3750 4250 60  0000 C CNN
-F 2 "bb:WS2818RGB" H 3750 4050 60  0001 C CNN
+F 2 "kbox:WS2818RGB" H 3750 4050 60  0001 C CNN
 F 3 "" H 3750 4050 60  0000 C CNN
 	1    3750 4000
@@
 F 0 "U15" H 3750 4550 60  0000 C CNN
 F 1 "NMEA_RGB" H 3750 5050 60  0000 C CNN
-F 2 "bb:WS2818RGB" H 3750 4850 60  0001 C CNN
+F 2 "kbox:WS2818RGB" H 3750 4850 60  0001 C CNN
 F 3 "" H 3750 4850 60  0000 C CNN
 	1    3750 4800
@@
 F 0 "U14" H 7250 4150 60  0000 C CNN
 F 1 "WIFI_RGB" H 7250 4650 60  0000 C CNN
-F 2 "bb:WS2818RGB" H 7250 4450 60  0001 C CNN
+F 2 "kbox:WS2818RGB" H 7250 4450 60  0001 C CNN
 F 3 "" H 7250 4450 60  0000 C CNN
 	1    7250 4400

Commit message: Preparing for macrofab
- Script to update values in kicad file
- Add MPN to parts that will be consigned
Parts:
- U13, U14, U15: PartNumber (none) -> WS2812RGB
Changed lines of the file:
@@
 F 2 "kbox:WS2818RGB" H 3750 4050 60  0001 C CNN
 F 3 "" H 3750 4050 60  0000 C CNN
+F 4 "WS2812RGB" H 3750 4000 60  0001 C CNN "PartNumber"
 	1    3750 4000
 	1    0    0    -1
@@
 F 2 "kbox:WS2818RGB" H 3750 4850 60  0001 C CNN
 F 3 "" H 3750 4850 60  0000 C CNN
+F 4 "WS2812RGB" H 3750 4800 60  0001 C CNN "PartNumber"
 	1    3750 4800
 	1    0    0    -1
@@
 F 2 "kbox:WS2818RGB" H 7250 4450 60  0001 C CNN
 F 3 "" H 7250 4450 60  0000 C CNN
+F 4 "WS2812RGB" H 7250 4400 60  0001 C CNN "PartNumber"
 	1    7250 4400
 	-1   0    0    -1
