File: sensors.sch (KiCad schematic (older format))
At the start: 12 parts, among them U10 BMP280, U11 BNO055

Commit message: More renaming from bb to kbox
Parts:
- U10: footprint bb:BMP280 -> kbox:BMP280
- U11: footprint bb:BNO055 -> kbox:BNO055
Changed lines of the file:
@@
 EESchema Schematic File Version 2
-LIBS:bb
+LIBS:kbox
 LIBS:power
 LIBS:device
@@
 LIBS:w_device
 LIBS:gsg-symbols
-LIBS:bb1-cache
+LIBS:kbox-cache
 EELAYER 25 0
 EELAYER END
@@
 F 0 "U10" H 2600 1800 60  0000 C CNN
 F 1 "BMP280" H 2300 1800 60  0000 C CNN
-F 2 "bb:BMP280" H 2400 1550 60  0001 C CNN
+F 2 "kbox:BMP280" H 2400 1550 60  0001 C CNN
 F 3 "" H 2400 1550 60  0000 C CNN
 F 4 "BMP280" H 2400 1550 60  0001 C CNN "PartNumber"
@@
 F 0 "U11" H 6700 2650 60  0000 C CNN
 F 1 "BNO055" H 7450 2200 60  0000 C CNN
-F 2 "bb:BNO055" H 6900 2350 60  0001 C CNN
+F 2 "kbox:BNO055" H 6900 2350 60  0001 C CNN
 F 3 "" H 6900 2350 60  0000 C CNN
 F 4 "BNO055" H 7500 2200 60  0001 C CNN "PartNumber"

Commit message: wip of v1d
Parts:
- C21: PartNumber CL10B682KB8SFNC -> CL10B682KB8WPNC
Changed lines of the file:
@@
 F 2 "Capacitors_SMD:C_0603" H 6800 1150 60  0001 C CNN
 F 3 "" H 6800 1150 60  0000 C CNN
-F 4 "CL10B682KB8SFNC" H 6800 1150 60  0001 C CNN "PartNumber"
+F 4 "CL10B682KB8WPNC" H 6800 1150 60  0001 C CNN "PartNumber"
 	1    6800 1150
 	-1   0    0    1
